Commit message: Update Package, remove wheels

File: description/robot_core.xacro (robot description, xacro)
@@ -31,5 +31,5 @@
         </visual>
     </link>
-    <joint name="wheel_fl_joint" type="continuous">
+    <!-- <joint name="wheel_fl_joint" type="continuous">
         <parent link="base_link"/>
         <child link="wheel_fl"/>
@@ -86,4 +86,4 @@
             <material name="black"/>
         </visual>
-    </link>
+    </link> -->
 </robot>
